File: KiCad/Metaldetector/Metaldetector.kicad_sch (KiCad schematic)
At the start: 0 parts

Commit message: QSPICE model er oprettet ikke done endu
Parts:
- added C1: C, symbol Device:C
- added L1: L, symbol Device:L
- added Q1, Q2: Q_NMOS, symbol Device:Q_NMOS
- added Q3: PMOS, symbol Simulation_SPICE:PMOS
- added R1: 10kR, symbol Device:R
- added R2: R, symbol Device:R
Connections:
- new net: C1.1, Q2.D, Q3.1 (D)
- new net: Q1.S, Q2.G, Q3.2 (G), R1.1
- new net: C1.2, L1.1
- new net: L1.2, R2.2
- new net +9V: Q1.D, Q3.3 (S)
- new net ARDUINO PWM: Q1.G
- new net GND: Q2.S, R1.2, R2.1
Other:
- note added: "D"
- note added: "G"
- note added: "S"

Commit message: Enkelte QSPICE ændringer plus kicad schematik af Hbro
Parts:
- removed C1: C, symbol Device:C
- removed L1: L, symbol Device:L
- removed Q1, Q2: Q_NMOS, symbol Device:Q_NMOS
- removed Q3: PMOS, symbol Simulation_SPICE:PMOS
- removed R1: 10kR, symbol Device:R
- removed R2: R, symbol Device:R
- added C4: 820n, symbol Device:C
- added R15: 45, symbol Device:R
- added Spole_conn1: Conn_01x02_Socket, symbol Connector:Conn_01x02_Socket
Connections:
- new net: C4.2, Spole_conn1.1 (Pin_1)
- new net: R15.1, Spole_conn1.2 (Pin_2)
- new net Højre side af H_Bro/Højre_out: R15.2
- new net Venstre side af H_Bro/Venstre_out: C4.1
Other:
- added sheet Dead time generator (dead_time.kicad_sch)
- added sheet Højre side af H_Bro (Højre_side.kicad_sch)
- added sheet Venstre side af H_Bro (Venstre_side.kicad_sch)
- note removed: "D"
- note removed: "G"
- note removed: "S"

Commit message: ændret kicad opsætning
Parts:
- removed C4: 820n, symbol Device:C
- removed R15: 45, symbol Device:R
- removed Spole_conn1: Conn_01x02_Socket, symbol Connector:Conn_01x02_Socket
Other:
- sheet Dead time generator: file dead_time.kicad_sch -> Dead_Time/Dead_Time.kicad_sch
- sheet Højre side af H_Bro: file Højre_side.kicad_sch -> Højre/Højre.kicad_sch
- sheet Højre side af H_Bro ports: added none; removed Højre_out
- sheet Venstre side af H_Bro: file Venstre_side.kicad_sch -> Venstre/Venstre.kicad_sch
- sheet Venstre side af H_Bro ports: added none; removed Venstre_out
