File: KiCad/Højre/Højre.kicad_sch (KiCad schematic)
At the start: 16 parts, among them Q1 NMOS_IRL530, Q3 NMOS_IRL530, Q5 NMOS_IRL530

Commit message: alla pcber er klar til routing
Parts:
- removed C1, C2_Load1: 820n, Capacitor_THT:C_Rect_L16.5mm_W8.7mm_P15.00mm_MKT, symbol Device:C
- removed C1_Load1: 100n, Capacitor_THT:C_Rect_L9.0mm_W2.5mm_P7.50mm_MKT, symbol Device:C
- removed C3_Load1: 2u2, Capacitor_THT:C_Rect_L24.0mm_W7.0mm_P22.50mm_MKT, symbol Device:C
- removed D1, D2: D, Diode_THT:D_DO-41_SOD81_P2.54mm_Vertical_AnodeUp, symbol Device:D
- removed Q1, Q3: NMOS_IRL530, Package_TO_SOT_THT:TO-220-3_Vertical, symbol Simulation_SPICE:NMOS
- removed R1, R3, R4: 1, Resistor_THT:R_Axial_DIN0204_L3.6mm_D1.6mm_P5.08mm_Horizontal, symbol Device:R
- removed R2: 1k, Resistor_THT:R_Axial_DIN0204_L3.6mm_D1.6mm_P5.08mm_Horizontal, symbol Device:R
- removed V_Inputs1: Conn_01x05_Pin, Connector_PinHeader_2.54mm:PinHeader_1x05_P2.54mm_Horizontal, symbol Connector:Conn_01x05_Pin
- removed V_Meas1: Conn_01x03_Pin, Connector_PinHeader_2.54mm:PinHeader_1x03_P2.54mm_Vertical, symbol Connector:Conn_01x03_Pin
- removed V_Out1: Conn_01x01_Pin, Connector_PinHeader_2.54mm:PinHeader_1x01_P2.54mm_Vertical, symbol Connector:Conn_01x01_Pin
- added C2: 820n, Capacitor_THT:C_Rect_L16.5mm_W8.7mm_P15.00mm_MKT, symbol Device:C
- added D3, D4: D, Diode_THT:D_DO-41_SOD81_P2.54mm_Vertical_AnodeUp, symbol Device:D
- added H_Input1: Conn_01x05_Pin, Connector_PinHeader_2.54mm:PinHeader_1x05_P2.54mm_Horizontal, symbol Connector:Conn_01x05_Pin
- added H_Out1: Conn_01x01_Pin, Connector_PinHeader_2.54mm:PinHeader_1x01_P2.54mm_Vertical, symbol Connector:Conn_01x01_Pin
- added Meas_H1: Conn_01x03_Pin, Connector_PinHeader_2.54mm:PinHeader_1x03_P2.54mm_Vertical, symbol Connector:Conn_01x03_Pin
- added Q4, Q6: NMOS_IRL530, Package_TO_SOT_THT:TO-220-3_Vertical, symbol Simulation_SPICE:NMOS
- added R5, R6, R8: 1, Resistor_THT:R_Axial_DIN0204_L3.6mm_D1.6mm_P5.08mm_Horizontal, symbol Device:R
- added R7: 1k, Resistor_THT:R_Axial_DIN0204_L3.6mm_D1.6mm_P5.08mm_Horizontal, symbol Device:R
- added R_Load1: 47, Connector_PinHeader_2.54mm:PinHeader_1x02_P2.54mm_Vertical, symbol Device:R
Connections:
- net +5V: now also D4.2 (A), H_Input1.5 (Pin_5)
- net +9V: now also H_Input1.1 (Pin_1), Q4.1 (D)
- net GND: now also H_Input1.4 (Pin_4), Q6.3 (S)
- net Meas_H_Out: now reaches Q5.1 (D)
- net Meas_H_Out: now also C2.2, D3.2 (A), Meas_H1.1 (Pin_1), Q4.3 (S), R_Load1.1
- net PWM2_NOT renamed Meas_GATE_M4
- net Meas_GATE_M4: now also Meas_H1.2 (Pin_2), R5.2
- new net: D3.1 (K), Q6.1 (D), R6.1, R7.2
- new net: D4.1 (K), R8.1
- new net: C2.1, R7.1, R8.2
- new net: H_Out1.1 (Pin_1), R_Load1.2
- new net Meas_GATE_M2: Meas_H1.3 (Pin_3), Q4.2 (G), R6.2
- new net PWM1_NOT: H_Input1.3 (Pin_3), Q6.2 (G)
- new net PWM2: H_Input1.2 (Pin_2), R5.1
