File: KiCad/Højre/Højre.kicad_pcb (KiCad board)
At the start: 2 copper layers, 66 x 57 mm, 14 parts, among them Q2 NMOS_IRL530, Q4 NMOS_IRL530, Q6 NMOS_IRL530

Commit message: gemme punkt før jeg laver om i deadtime pcb
Routing:
- net /Meas_GATE_M2: track 54.8 -> 60.9 mm
- net /Meas_H_Out: track 73.3 -> 75.5 mm
- net /PWM2: track 45.2 -> 46.5 mm
- net Net-(C2-Pad1): track 22.8 -> 24.0 mm
- net /PWM1_NOT: track 10.2 -> 10.9 mm
- net /Meas_GATE_M4: track 33.4 -> 34.0 mm
Changed lines of the file:
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@@
 	)
 	(segment
-		(start 166 109.96)
-		(end 158.622735 109.96)
+		(start 157.54 109.96)
+		(end 148.8 118.7)
 		(width 0.8)
 		(layer "B.Cu")
@@
 	)
 	(segment
-		(start 144 123.25)
-		(end 145.75 121.5)
-		(width 0.8)
-		(layer "B.Cu")
-		(net 1)
-	)
-	(segment
-		(start 149.832735 118.75)
-		(end 148.8 118.75)
+		(start 153.5 134)
+		(end 149.25 134)
+		(width 0.8)
+		(layer "B.Cu")
+		(net 1)
+	)
+	(segment
+		(start 142.75 127.5)
+		(end 142.75 123.25)
 		(width 0.8)
 		(layer "B.Cu")
@@
 	)
 	(segment
-		(start 145.75 121.5)
-		(end 148.8 121.5)
-		(width 0.8)
-		(layer "B.Cu")
-		(net 1)
-	)
-	(segment
-		(start 153.5 134)
-		(end 150 134)
-		(width 0.8)
-		(layer "B.Cu")
-		(net 1)
-	)
-	(segment
-		(start 144 128)
-		(end 144 123.25)
+		(start 149.25 134)
+		(end 142.75 127.5)
 		(width 0.8)
 		(layer "B.Cu")
@@
 	)
 	(segment
-		(start 158.622735 109.96)
-		(end 149.832735 118.75)
+		(start 144.5 121.5)
+		(end 148.8 121.5)
+		(width 0.8)
+		(layer "B.Cu")
+		(net 1)
+	)
+	(segment
+		(start 166 109.96)
+		(end 157.54 109.96)
+		(width 0.8)
+		(layer "B.Cu")
+		(net 1)
+	)
+	(segment
+		(start 148.8 118.7)
+		(end 148.8 118.75)
+		(width 0.8)
+		(layer "B.Cu")
+		(net 1)
+	)
+	(segment
+		(start 142.75 123.25)
+		(end 144.5 121.5)
 		(width 0.8)
 		(layer "B.Cu")
@@
 	)
 	(segment
-		(start 150 134)
-		(end 144 128)
-		(width 0.8)
-		(layer "B.Cu")
-		(net 1)
-	)
-	(segment
-		(start 167.292266 105.519)
-		(end 167.269 105.519)
-		(width 0.8)
-		(layer "B.Cu")
-		(net 2)
-	)
-	(segment
-		(start 159.5 112.5)
-		(end 166.25 112.5)
-		(width 0.8)
-		(layer "B.Cu")
-		(net 2)
-	)
-	(segment
-		(start 167.901 106.151)
-		(end 167.901 106.127734)
+		(start 168.75 106)
+		(end 168.75 111)
 		(width 0.8)
 		(layer "B.Cu")
@@
 	)
 	(segment
-		(start 167.901 106.127734)
-		(end 167.292266 105.519)
+		(start 167.25 112.5)
+		(end 159.5 112.5)
 		(width 0.8)
 		(layer "B.Cu")
@@
 	)
 	(segment
-		(start 166.25 112.5)
-		(end 168 110.75)
-		(width 0.8)
-		(layer "B.Cu")
-		(net 2)
-	)
-	(segment
-		(start 168 106.25)
-		(end 167.901 106.151)
-		(width 0.8)
-		(layer "B.Cu")
-		(net 2)
-	)
-	(segment
-		(start 165.96 104.21)
-		(end 165.96 102.34)
-		(width 0.8)
-		(layer "B.Cu")
-		(net 2)
-	)
-	(segment
-		(start 167.269 105.519)
-		(end 165.96 104.21)
-		(width 0.8)
-		(layer "B.Cu")
-		(net 2)
-	)
-	(segment
-		(start 168 110.75)
-		(end 168 106.25)
+		(start 168.75 111)
+		(end 167.25 112.5)
+		(width 0.8)
+		(layer "B.Cu")
+		(net 2)
+	)
+	(segment
+		(start 165.96 102.34)
+		(end 165.96 103.21)
+		(width 0.8)
+		(layer "B.Cu")
+		(net 2)
+	)
+	(segment
+		(start 165.96 103.21)
+		(end 168.75 106)
 		(width 0.8)
 		(layer "B.Cu")
@@
 	)
 	(segment
+		(start 169.04 117.46)
+		(end 174 112.5)
+		(width 0.8)
+		(layer "B.Cu")
+		(net 7)
+	)
+	(segment
+		(start 171 92)
+		(end 159 92)
+		(width 0.8)
+		(layer "B.Cu")
+		(net 7)
+	)
+	(segment
+		(start 174 112.5)
+		(end 174 95)
+		(width 0.8)
+		(layer "B.Cu")
+		(net 7)
+	)
+	(segment
+		(start 159 92)
+		(end 156.96 94.04)
+		(width 0.8)
+		(layer "B.Cu")
+		(net 7)
+	)
+	(segment
 		(start 167.75 117.46)
 		(end 169.04 117.46)
@@
 	)
 	(segment
-		(start 173.5 94.5)
+		(start 174 95)
 		(end 171 92)
 		(width 0.8)
@@
 	)
 	(segment
-		(start 157.165133 95.635)
+		(start 156.96 94.04)
 		(end 156.96 95.635)
 		(width 0.8)
@@
 	)
 	(segment
-		(start 169.04 117.46)
-		(end 173.5 113)
-		(width 0.8)
-		(layer "B.Cu")
-		(net 7)
-	)
-	(segment
-		(start 173.5 113)
-		(end 173.5 94.5)
-		(width 0.8)
-		(layer "B.Cu")
-		(net 7)
-	)
-	(segment
-		(start 171 92)
-		(end 160.800133 92)
-		(width 0.8)
-		(layer "B.Cu")
-		(net 7)
-	)
-	(segment
-		(start 160.800133 92)
-		(end 157.165133 95.635)
-		(width 0.8)
-		(layer "B.Cu")
-		(net 7)
+		(start 153.599 98.401)
+		(end 157.849 98.401)
+		(width 0.8)
+		(layer "B.Cu")
+		(net 8)
+	)
+	(segment
+		(start 152.21 99.79)
+		(end 153.599 98.401)
+		(width 0.8)
+		(layer "B.Cu")
+		(net 8)
+	)
+	(segment
+		(start 152.21 101.05)
+		(end 152.21 99.79)
+		(width 0.8)
+		(layer "B.Cu")
+		(net 8)
 	)
 	(segment
@@
 	)
 	(segment
-		(start 152.21 101.05)
-		(end 154.859 98.401)
-		(width 0.8)
-		(layer "B.Cu")
-		(net 8)
-	)
-	(segment
-		(start 154.859 98.401)
-		(end 157.849 98.401)
-		(width 0.8)
-		(layer "B.Cu")
-		(net 8)
-	)
-	(segment
 		(start 154.42 95.635)
 		(end 152.365 95.635)
@@
 	)
 	(segment
+		(start 167.75 127.5)
+		(end 167.75 122.54)
+		(width 0.8)
+		(layer "B.Cu")
+		(net 11)
+	)
+	(segment
+		(start 163.25 132)
+		(end 167.75 127.5)
+		(width 0.8)
+		(layer "B.Cu")
+		(net 11)
+	)
+	(segment
+		(start 156 132.25)
+		(end 156.25 132)
+		(width 0.8)
+		(layer "B.Cu")
+		(net 11)
+	)
+	(segment
 		(start 156 133.96)
 		(end 156 132.25)
@@
 	)
 	(segment
-		(start 152.16 132.25)
-		(end 156 132.25)
+		(start 146.21 127.335)
+		(end 150.875 132)
+		(width 0.8)
+		(layer "B.Cu")
+		(net 11)
+	)
+	(segment
+		(start 150.875 132)
+		(end 155.75 132)
 		(width 0.8)
 		(layer "B.Cu")
@@
 	)
 	(segment
+		(start 156.25 132)
+		(end 163.25 132)
+		(width 0.8)
+		(layer "B.Cu")
+		(net 11)
+	)
+	(segment
 		(start 146.21 126.3)
-		(end 152.16 132.25)
-		(width 0.8)
-		(layer "B.Cu")
-		(net 11)
-	)
-	(segment
-		(start 156 132.25)
-		(end 163 132.25)
-		(width 0.8)
-		(layer "B.Cu")
-		(net 11)
-	)
-	(segment
-		(start 163 132.25)
-		(end 167.75 127.5)
-		(width 0.8)
-		(layer "B.Cu")
-		(net 11)
-	)
-	(segment
-		(start 167.75 127.5)
-		(end 167.75 122.54)
-		(width 0.8)
-		(layer "B.Cu")
-		(net 11)
+		(end 146.21 127.335)
+		(width 0.8)
+		(layer "B.Cu")
+		(net 11)
+	)
+	(segment
+		(start 155.75 132)
+		(end 156 132.25)
+		(width 0.8)
+		(layer "B.Cu")
+		(net 11)
+	)
+	(segment
+		(start 156 138.5)
+		(end 148.75 138.5)
+		(width 0.8)
+		(layer "B.Cu")
+		(net 12)
+	)
+	(segment
+		(start 144.58 107.42)
+		(end 148.8 107.42)
+		(width 0.8)
+		(layer "B.Cu")
+		(net 12)
+	)
+	(segment
+		(start 137.25 114.75)
+		(end 144.58 107.42)
+		(width 0.8)
+		(layer "B.Cu")
+		(net 12)
+	)
+	(segment
+		(start 148.75 138.5)
+		(end 137.25 127)
+		(width 0.8)
+		(layer "B.Cu")
+		(net 12)
 	)
 	(segment
@@
 	)
 	(segment
-		(start 149.75 136.25)
-		(end 138.75 125.25)
-		(width 0.8)
-		(layer "B.Cu")
-		(net 12)
-	)
-	(segment
-		(start 146.33 107.42)
-		(end 148.8 107.42)
-		(width 0.8)
-		(layer "B.Cu")
-		(net 12)
-	)
-	(segment
 		(start 158.58 134)
 		(end 158.58 135.92)
@@
 	)
 	(segment
-		(start 158.25 136.25)
-		(end 149.75 136.25)
-		(width 0.8)
-		(layer "B.Cu")
-		(net 12)
-	)
-	(segment
 		(start 158.58 135.92)
-		(end 158.25 136.25)
-		(width 0.8)
-		(layer "B.Cu")
-		(net 12)
-	)
-	(segment
-		(start 138.75 125.25)
-		(end 138.75 115)
-		(width 0.8)
-		(layer "B.Cu")
-		(net 12)
-	)
-	(segment
-		(start 138.75 115)
-		(end 146.33 107.42)
-		(width 0.8)
-		(layer "B.Cu")
+		(end 156 138.5)
+		(width 0.8)
+		(layer "B.Cu")
+		(net 12)
+	)
+	(segment
+		(start 137.25 127)
+		(end 137.25 114.75)
+		(width 0.8)
+		(layer "B.Cu")
