File: KiCad/Venstre/Venstre.kicad_sch (KiCad schematic)
At the start: 14 parts, among them Q2 NMOS_IRL530, Q4 NMOS_IRL530, Q6 NMOS_IRL530

Commit message: alla pcber er klar til routing
Parts:
- removed C2: 820n, Capacitor_THT:C_Rect_L16.5mm_W8.7mm_P15.00mm_MKT, symbol Device:C
- removed D3, D4: D, Diode_THT:D_DO-41_SOD81_P2.54mm_Vertical_AnodeUp, symbol Device:D
- removed H_Input1: Conn_01x05_Pin, Connector_PinHeader_2.54mm:PinHeader_1x05_P2.54mm_Horizontal, symbol Connector:Conn_01x05_Pin
- removed H_Out1: Conn_01x01_Pin, Connector_PinHeader_2.54mm:PinHeader_1x01_P2.54mm_Vertical, symbol Connector:Conn_01x01_Pin
- removed Meas_H1: Conn_01x03_Pin, Connector_PinHeader_2.54mm:PinHeader_1x03_P2.54mm_Vertical, symbol Connector:Conn_01x03_Pin
- removed Q4, Q6: NMOS_IRL530, Package_TO_SOT_THT:TO-220-3_Vertical, symbol Simulation_SPICE:NMOS
- removed R5, R7, R8: 1, Resistor_THT:R_Axial_DIN0204_L3.6mm_D1.6mm_P5.08mm_Horizontal, symbol Device:R
- removed R6: 1k, Resistor_THT:R_Axial_DIN0204_L3.6mm_D1.6mm_P5.08mm_Horizontal, symbol Device:R
- removed R_Load1: 47, Connector_PinHeader_2.54mm:PinHeader_1x02_P2.54mm_Vertical, symbol Device:R
- added C1, C2_Load1: 820n, Capacitor_THT:C_Rect_L16.5mm_W8.7mm_P15.00mm_MKT, symbol Device:C
- added C1_Load1: 100n, Capacitor_THT:C_Rect_L9.0mm_W2.5mm_P7.50mm_MKT, symbol Device:C
- added C3_Load1: 2u2, Capacitor_THT:C_Rect_L24.0mm_W7.0mm_P22.50mm_MKT, symbol Device:C
- added D1, D2: D, Diode_THT:D_DO-41_SOD81_P2.54mm_Vertical_AnodeUp, symbol Device:D
- added Q1, Q3: NMOS_IRL530, Package_TO_SOT_THT:TO-220-3_Vertical, symbol Simulation_SPICE:NMOS
- added R1, R3, R4: 1, Resistor_THT:R_Axial_DIN0204_L3.6mm_D1.6mm_P5.08mm_Horizontal, symbol Device:R
- added R2: 1k, Resistor_THT:R_Axial_DIN0204_L3.6mm_D1.6mm_P5.08mm_Horizontal, symbol Device:R
- added V_Inputs1: Conn_01x05_Pin, Connector_PinHeader_2.54mm:PinHeader_1x05_P2.54mm_Horizontal, symbol Connector:Conn_01x05_Pin
- added V_Meas1: Conn_01x03_Pin, Connector_PinHeader_2.54mm:PinHeader_1x03_P2.54mm_Vertical, symbol Connector:Conn_01x03_Pin
- added V_Out1: Conn_01x01_Pin, Connector_PinHeader_2.54mm:PinHeader_1x01_P2.54mm_Vertical, symbol Connector:Conn_01x01_Pin
Connections:
- net +5V: now also D1.2 (A), V_Inputs1.5 (Pin_5)
- net +9V: now also V_Inputs1.1 (Pin_1)
- net GND: now also Q1.3 (S), Q3.3 (S), V_Inputs1.4 (Pin_4)
- net Meas_GATE_M2 renamed Meas_GATE_M1
- net Meas_GATE_M1: now also R3.2, V_Meas1.3 (Pin_3)
- net Meas_H_Out renamed Meas_V_Out
- net Meas_V_Out: now also C1.2, C1_Load1.1, C2_Load1.2, C3_Load1.1, D2.2 (A), Q3.1 (D), V_Meas1.1 (Pin_1)
- new net: C1_Load1.2, C2_Load1.1, C3_Load1.2, V_Out1.1 (Pin_1)
- new net: C1.1, R1.2, R2.1
- new net: D1.1 (K), R1.1
- new net: D2.1 (K), Q1.1 (D), R2.2, R3.1
- new net Meas_GATE_M3: Q3.2 (G), R4.2, V_Meas1.2 (Pin_2)
- new net PWM1: R4.1, V_Inputs1.2 (Pin_2)
- new net PWM2_NOT: Q1.2 (G), V_Inputs1.3 (Pin_3)
