File: KiCad/Venstre/Venstre.kicad_pcb (KiCad board)
At the start: 2 copper layers, 66 x 57 mm, 16 parts, among them Q1 NMOS_IRL530, Q3 NMOS_IRL530, Q5 NMOS_IRL530

Commit message: gemme punkt før jeg laver om i deadtime pcb
Routing:
- net /Meas_V_Out: track 94.8 -> 91.2 mm
- net /Meas_GATE_M1: track 70.3 -> 72.7 mm
- net /Meas_GATE_M3: track 32.8 -> 34.3 mm
- net /PWM2_NOT: track 9.08 -> 10.4 mm
- net /PWM1: track 45.6 -> 46.8 mm
Changed lines of the file:
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@@
 	)
 	(segment
-		(start 152.79 109.91)
-		(end 156.04 109.91)
+		(start 144.5375 95.66)
+		(end 148.79 95.66)
 		(width 0.8)
 		(layer "B.Cu")
@@
 	)
 	(segment
-		(start 146.415 98.16)
-		(end 151.29 98.16)
+		(start 139.7475 90.87)
+		(end 144.5375 95.66)
 		(width 0.8)
 		(layer "B.Cu")
@@
 	)
 	(segment
+		(start 151.04 114.91)
+		(end 156.04 109.91)
+		(width 0.8)
+		(layer "B.Cu")
+		(net 1)
+	)
+	(segment
+		(start 144.29 114.91)
+		(end 151.04 114.91)
+		(width 0.8)
+		(layer "B.Cu")
+		(net 1)
+	)
+	(segment
 		(start 148.79 93.41)
 		(end 148.79 95.66)
@@
 	)
 	(segment
-		(start 131.79 90.87)
-		(end 139.125 90.87)
-		(width 0.8)
-		(layer "B.Cu")
-		(net 1)
-	)
-	(segment
-		(start 139.125 90.87)
-		(end 146.415 98.16)
-		(width 0.8)
-		(layer "B.Cu")
-		(net 1)
-	)
-	(segment
-		(start 144.29 114.91)
-		(end 147.79 114.91)
-		(width 0.8)
-		(layer "B.Cu")
-		(net 1)
-	)
-	(segment
 		(start 151.29 100.91)
 		(end 148.79 100.91)
@@
 	)
 	(segment
-		(start 147.79 114.91)
-		(end 152.79 109.91)
+		(start 131.79 90.87)
+		(end 139.7475 90.87)
 		(width 0.8)
 		(layer "B.Cu")
@@
 	)
 	(segment
+		(start 143.04 83.21)
+		(end 143.04 81.96)
+		(width 0.8)
+		(layer "B.Cu")
+		(net 4)
+	)
+	(segment
 		(start 138.75 88.33)
-		(end 143.04 84.04)
+		(end 138.75 87.5)
 		(width 0.8)
 		(layer "B.Cu")
@@
 	)
 	(segment
-		(start 143.04 84.04)
-		(end 143.04 81.96)
+		(start 138.75 87.5)
+		(end 143.04 83.21)
 		(width 0.8)
 		(layer "B.Cu")
@@
 	)
 	(segment
+		(start 162.33 88.33)
+		(end 167.5 93.5)
+		(width 0.8)
+		(layer "B.Cu")
+		(net 7)
+	)
+	(segment
+		(start 143.83 88.33)
+		(end 148.79 88.33)
+		(width 0.8)
+		(layer "B.Cu")
+		(net 7)
+	)
+	(segment
+		(start 148.79 88.33)
+		(end 162.33 88.33)
+		(width 0.8)
+		(layer "B.Cu")
+		(net 7)
+	)
+	(segment
 		(start 139.21 116.58)
 		(end 139.21 114.91)
@@
 	)
 	(segment
-		(start 143.83 88.33)
-		(end 148.79 88.33)
-		(width 0.8)
-		(layer "B.Cu")
-		(net 7)
-	)
-	(segment
-		(start 166.29 93.91)
-		(end 166.29 105.66)
-		(width 0.8)
-		(layer "B.Cu")
-		(net 7)
-	)
-	(segment
-		(start 154.79 117.16)
-		(end 139.79 117.16)
-		(width 0.8)
-		(layer "B.Cu")
-		(net 7)
-	)
-	(segment
-		(start 148.79 88.33)
-		(end 160.71 88.33)
-		(width 0.8)
-		(layer "B.Cu")
-		(net 7)
-	)
-	(segment
-		(start 139.79 117.16)
+		(start 167.5 93.5)
+		(end 167.5 104.45)
+		(width 0.8)
+		(layer "B.Cu")
+		(net 7)
+	)
+	(segment
+		(start 154.2 117.75)
+		(end 140.38 117.75)
+		(width 0.8)
+		(layer "B.Cu")
+		(net 7)
+	)
+	(segment
+		(start 167.5 104.45)
+		(end 154.2 117.75)
+		(width 0.8)
+		(layer "B.Cu")
+		(net 7)
+	)
+	(segment
+		(start 140.38 117.75)
 		(end 139.21 116.58)
 		(width 0.8)
@@
 	)
 	(segment
-		(start 160.71 88.33)
-		(end 166.29 93.91)
-		(width 0.8)
-		(layer "B.Cu")
-		(net 7)
-	)
-	(segment
-		(start 166.29 105.66)
-		(end 154.79 117.16)
-		(width 0.8)
-		(layer "B.Cu")
-		(net 7)
+		(start 148.79 79.91)
+		(end 148.79 83.66)
+		(width 0.8)
+		(layer "B.Cu")
+		(net 8)
+	)
+	(segment
+		(start 146.54 77.66)
+		(end 148.79 79.91)
+		(width 0.8)
+		(layer "B.Cu")
+		(net 8)
 	)
 	(segment
 		(start 147.29 85.16)
-		(end 144.04 85.16)
-		(width 0.8)
-		(layer "B.Cu")
-		(net 8)
-	)
-	(segment
-		(start 141.54 87.66)
+		(end 143.59 85.16)
+		(width 0.8)
+		(layer "B.Cu")
+		(net 8)
+	)
+	(segment
+		(start 141.54 88.91)
+		(end 143.5 90.87)
+		(width 0.8)
+		(layer "B.Cu")
+		(net 8)
+	)
+	(segment
+		(start 141.54 87.21)
 		(end 141.54 88.91)
 		(width 0.8)
@@
 	)
 	(segment
-		(start 144.04 85.16)
-		(end 141.54 87.66)
+		(start 143.59 85.16)
+		(end 141.54 87.21)
 		(width 0.8)
 		(layer "B.Cu")
@@
 	)
 	(segment
-		(start 148.79 79.91)
-		(end 148.79 83.66)
-		(width 0.8)
-		(layer "B.Cu")
-		(net 8)
-	)
-	(segment
-		(start 146.54 77.66)
-		(end 148.79 79.91)
-		(width 0.8)
-		(layer "B.Cu")
-		(net 8)
-	)
-	(segment
-		(start 141.54 88.91)
-		(end 143.5 90.87)
-		(width 0.8)
-		(layer "B.Cu")
-		(net 8)
-	)
-	(segment
 		(start 141.75 114.91)
 		(end 141.79 114.87)
@@
 	)
 	(segment
+		(start 130.04 103.45)
+		(end 130.04 108.41)
+		(width 0.8)
+		(layer "B.Cu")
+		(net 9)
+	)
+	(segment
+		(start 141.38 112.75)
+		(end 141.79 113.16)
+		(width 0.8)
+		(layer "B.Cu")
+		(net 9)
+	)
+	(segment
+		(start 130.04 108.41)
+		(end 134.38 112.75)
+		(width 0.8)
+		(layer "B.Cu")
+		(net 9)
+	)
+	(segment
+		(start 134.38 112.75)
+		(end 141.38 112.75)
+		(width 0.8)
+		(layer "B.Cu")
+		(net 9)
+	)
+	(segment
+		(start 151.58 109.42)
+		(end 151.58 107.21)
+		(width 0.8)
+		(layer "B.Cu")
+		(net 9)
+	)
+	(segment
+		(start 141.79 113.16)
+		(end 142.2 112.75)
+		(width 0.8)
+		(layer "B.Cu")
+		(net 9)
+	)
+	(segment
+		(start 142.2 112.75)
+		(end 148.25 112.75)
+		(width 0.8)
+		(layer "B.Cu")
+		(net 9)
+	)
+	(segment
+		(start 141.79 113.16)
+		(end 141.975 112.975)
+		(width 0.8)
+		(layer "B.Cu")
+		(net 9)
+	)
+	(segment
+		(start 141.75 114.91)
+		(end 141.79 114.87)
+		(width 0.8)
+		(layer "B.Cu")
+		(net 9)
+	)
+	(segment
+		(start 148.25 112.75)
+		(end 151.58 109.42)
+		(width 0.8)
+		(layer "B.Cu")
+		(net 9)
+	)
+	(segment
 		(start 141.79 114.87)
 		(end 141.79 113.16)
@@
 	)
 	(segment
-		(start 141.79 113.16)
-		(end 145.63 113.16)
-		(width 0.8)
-		(layer "B.Cu")
-		(net 9)
-	)
-	(segment
-		(start 134.79 113.16)
-		(end 141.79 113.16)
-		(width 0.8)
-		(layer "B.Cu")
-		(net 9)
-	)
-	(segment
-		(start 145.63 113.16)
-		(end 151.58 107.21)
-		(width 0.8)
-		(layer "B.Cu")
-		(net 9)
-	)
-	(segment
-		(start 141.75 114.91)
-		(end 141.79 114.87)
-		(width 0.8)
-		(layer "B.Cu")
-		(net 9)
-	)
-	(segment
-		(start 130.04 108.41)
-		(end 134.79 113.16)
-		(width 0.8)
-		(layer "B.Cu")
-		(net 9)
-	)
-	(segment
-		(start 130.04 103.45)
-		(end 130.04 108.41)
-		(width 0.8)
-		(layer "B.Cu")
-		(net 9)
-	)
-	(segment
-		(start 143.779 80.159)
-		(end 143.779 80.149)
+		(start 144.5 79.75)
+		(end 139.25 79.75)
 		(width 0.8)
 		(layer "B.Cu")
@@
 	)
 	(segment
-		(start 139.941 79.311)
+		(start 145.58 80.83)
+		(end 144.5 79.75)
+		(width 0.8)
+		(layer "B.Cu")
+		(net 11)
+	)
+	(segment
+		(start 138.29 78.79)
 		(end 138.29 77.66)
 		(width 0.8)
@@
 	)
 	(segment
+		(start 139.25 79.75)
+		(end 138.29 78.79)
+		(width 0.8)
+		(layer "B.Cu")
+		(net 11)
+	)
+	(segment
 		(start 145.58 81.96)
-		(end 143.779 80.159)
+		(end 145.58 80.83)
 		(width 0.8)
 		(layer "B.Cu")
@@
 	)
 	(segment
-		(start 143.779 80.149)
-		(end 142.941 79.311)
-		(width 0.8)
-		(layer "B.Cu")
-		(net 11)
-	)
-	(segment
-		(start 142.941 79.311)
-		(end 139.941 79.311)
-		(width 0.8)
-		(layer "B.Cu")
-		(net 11)
-	)
-	(segment
-		(start 136.08 72.91)
-		(end 126.79 72.91)
+		(start 123.25 76)
+		(end 123.25 92.87)
 		(width 0.8)
 		(layer "B.Cu")
@@
 	)
 	(segment
-		(start 126.79 72.91)
-		(end 124.29 75.41)
+		(start 126.34 72.91)
+		(end 123.25 76)
 		(width 0.8)
 		(layer "B.Cu")
@@
 	)
 	(segment
-		(start 124.29 75.41)
-		(end 124.29 93.91)
-		(width 0.8)
-		(layer "B.Cu")
-		(net 12)
-	)
-	(segment
-		(start 124.29 93.91)
+		(start 123.25 92.87)
 		(end 128.75 98.37)
 		(width 0.8)
@@
 		(width 0.8)
 		(layer "B.Cu")
+		(net 12)
+	)
+	(segment
+		(start 136.08 72.91)
+		(end 126.34 72.91)
+		(width 0.8)
+		(layer "B.Cu")
