File: KiCad/rx forstærker/rx forstærker.kicad_sch (KiCad schematic)
At the start: 12 parts, among them J1 Rx spole, J2 Pot_pins, J4 MALE Headers, U1 MCP6002-xMC

Commit message: lavet pcb design til arduino/Rx forstærker
Parts:
- C1_DC_protect1: renamed from C1_DC_protect; footprint (none) -> Capacitor_THT:C_Rect_L7.0mm_W2.0mm_P5.00mm
- C2_DC_protect1: renamed from C2_DC_protect; footprint (none) -> Capacitor_THT:C_Rect_L7.0mm_W2.0mm_P5.00mm
- C3: footprint (none) -> Capacitor_THT:C_Rect_L16.5mm_W8.7mm_P15.00mm_MKT
- I2C_skærm_FEMALE_4xpin1: renamed from I2C_skærm_MALE_headers; footprint (none) -> Connector_PinHeader_2.54mm:PinHeader_1x04_P2.54mm_Vertical
- J1: footprint (none) -> Connector_PinHeader_2.54mm:PinHeader_1x02_P2.54mm_Vertical
- J2: value Pot_pins -> Pot_pins_2xpin; footprint (none) -> Connector_PinHeader_2.54mm:PinHeader_1x02_P2.54mm_Vertical
- J4: value MALE Headers -> MALE Headers 5xpin; footprint (none) -> Connector_PinHeader_2.54mm:PinHeader_2x05_P2.54mm_Vertical
- R1, R1,2, R2: footprint (none) -> Resistor_THT:R_Axial_DIN0411_L9.9mm_D3.6mm_P20.32mm_Horizontal
- U1: footprint Package_DFN_QFN:DFN-8-1EP_3x2mm_P0.5mm_EP1.75x1.45mm -> Package_DIP:DIP-8_W7.62mm
Changed lines of the file:
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@@
 (kicad_sch
-	(version 20231120)
+	(version 20250114)
 	(generator "eeschema")
-	(generator_version "8.0")
+	(generator_version "9.0")
 	(paper "A4")
 	(junction
@@
 	)
 	(junction
+		(at 166.37 125.73)
+		(diameter 0)
+		(color 0 0 0 0)
+	)
+	(junction
+		(at 160.02 138.43)
+		(diameter 0)
+		(color 0 0 0 0)
+	)
+	(junction
 		(at 81.28 99.06)
 		(diameter 0)
@@
 	(label "PA_power_off"
 		(at 191.77 102.87 0)
-		(fields_autoplaced yes)
 		(effects
 			(font
@@
 	(label "TX_out->PA"
 		(at 191.77 100.33 0)
-		(fields_autoplaced yes)
 		(effects
 			(font
@@
 	(label "SCL"
 		(at 193.04 67.31 0)
-		(fields_autoplaced yes)
 		(effects
 			(font
@@
 	(label "Vin"
 		(at 193.04 72.39 0)
-		(fields_autoplaced yes)
 		(effects
 			(font
@@
 	(label "2.5V"
 		(at 104.14 99.06 0)
-		(fields_autoplaced yes)
 		(effects
 			(font
@@
 	(label "Debug"
 		(at 191.77 105.41 0)
-		(fields_autoplaced yes)
 		(effects
 			(font
@@
 	(label "Start{slash}Stop"
 		(at 191.77 110.49 0)
-		(fields_autoplaced yes)
 		(effects
 			(font
@@
 	(label "Rx_ADC "
 		(at 143.51 100.33 0)
-		(fields_autoplaced yes)
 		(effects
 			(font
@@
 	(label "Kalibrering"
 		(at 191.77 107.95 0)
-		(fields_autoplaced yes)
 		(effects
 			(font
@@
 	(label "rx spole. 12.225mH og 71 ohm"
 		(at 44.45 99.06 0)
-		(fields_autoplaced yes)
 		(effects
 			(font
@@
 	(label "GND"
 		(at 193.04 69.85 0)
-		(fields_autoplaced yes)
 		(effects
 			(font
@@
 	(label "SDA"
 		(at 193.04 64.77 0)
-		(fields_autoplaced yes)
 		(effects
 			(font
@@
 			)
 		)
-		(property "Footprint" "Package_DFN_QFN:DFN-8-1EP_3x2mm_P0.5mm_EP1.75x1.45mm"
+		(property "Footprint" "Package_DIP:DIP-8_W7.62mm"
 			(at 128.27 101.6 0)
 			(effects
@@
 			)
 		)
-		(property "Footprint" ""
+		(property "Footprint" "Resistor_THT:R_Axial_DIN0411_L9.9mm_D3.6mm_P20.32mm_Horizontal"
 			(at 102.362 91.44 90)
 			(effects
@@
 			)
 		)
-		(property "Value" "Pot_pins"
+		(property "Value" "Pot_pins_2xpin"
 			(at 129.54 116.2049 90)
 			(effects
@@
 			)
 		)
-		(property "Footprint" ""
+		(property "Footprint" "Connector_PinHeader_2.54mm:PinHeader_1x02_P2.54mm_Vertical"
 			(at 128.27 116.84 0)
 			(effects
@@
 			)
 		)
-		(property "Footprint" ""
+		(property "Footprint" "Connector_PinHeader_2.54mm:PinHeader_1x02_P2.54mm_Vertical"
 			(at 39.37 99.06 0)
 			(effects
@@
 		(dnp no)
 		(fields_autoplaced yes)
-		(property "Reference" "C1_DC_protect"
+		(property "Reference" "C1_DC_protect1"
 			(at 92.71 91.44 90)
 			(effects
@@
 			)
 		)
-		(property "Footprint" ""
+		(property "Footprint" "Capacitor_THT:C_Rect_L7.0mm_W2.0mm_P5.00mm"
 			(at 96.52 98.0948 0)
 			(effects
@@
 			(project ""
 				(path "/5c43024a-135c-49bd-9b6f-adf795041e03"
-					(reference "C1_DC_protect")
+					(reference "C1_DC_protect1")
 					(unit 1)
 				)
@@
 			)
 		)
-		(property "Footprint" ""
+		(property "Footprint" "Resistor_THT:R_Axial_DIN0411_L9.9mm_D3.6mm_P20.32mm_Horizontal"
 			(at 122.428 118.11 90)
 			(effects
@@
 			)
 		)
-		(property "Footprint" ""
+		(property "Footprint" "Resistor_THT:R_Axial_DIN0411_L9.9mm_D3.6mm_P20.32mm_Horizontal"
 			(at 102.362 106.68 90)
 			(effects
@@
 			)
 		)
-		(property "Value" "MALE Headers"
+		(property "Value" "MALE Headers 5xpin"
 			(at 210.82 105.41 0)
 			(effects
@@
 			)
 		)
-		(property "Footprint" ""
+		(property "Footprint" "Connector_PinHeader_2.54mm:PinHeader_2x05_P2.54mm_Vertical"
 			(at 209.55 105.41 0)
 			(effects
@@
 		(on_board yes)
 		(dnp no)
-		(property "Reference" "C2_DC_protect"
+		(property "Reference" "C2_DC_protect1"
 			(at 123.444 129.032 0)
 			(effects
@@
 			)
 		)
-		(property "Footprint" ""
+		(property "Footprint" "Capacitor_THT:C_Rect_L7.0mm_W2.0mm_P5.00mm"
 			(at 119.6848 123.19 0)
 			(effects
@@
 			(project "rx forstærker"
 				(path "/5c43024a-135c-49bd-9b6f-adf795041e03"
-					(reference "C2_DC_protect")
+					(reference "C2_DC_protect1")
 					(unit 1)
 				)
@@
 			)
 		)
-		(property "Footprint" ""
+		(property "Footprint" "Capacitor_THT:C_Rect_L16.5mm_W8.7mm_P15.00mm_MKT"
 			(at 82.2452 114.3 0)
 			(effects
@@
 	)
 	(symbol
+		(lib_id "power:PWR_FLAG")
+		(at 160.02 138.43 270)
+		(unit 1)
+		(exclude_from_sim no)
+		(in_bom yes)
+		(on_board yes)
+		(dnp no)
+		(fields_autoplaced yes)
+		(property "Reference" "#FLG02"
+			(at 161.925 138.43 0)
+			(effects
+				(font
+					(size 1.27 1.27)
+				)
+				(hide yes)
+			)
+		)
+		(property "Value" "PWR_FLAG"
+			(at 163.83 138.4299 90)
+			(effects
+				(font
+					(size 1.27 1.27)
+				)
+				(justify left)
+			)
+		)
+		(property "Footprint" ""
+			(at 160.02 138.43 0)
+			(effects
+				(font
+					(size 1.27 1.27)
+				)
+				(hide yes)
+			)
+		)
+		(property "Datasheet" "~"
+			(at 160.02 138.43 0)
+			(effects
+				(font
+					(size 1.27 1.27)
+				)
+				(hide yes)
+			)
+		)
+		(property "Description" "Special symbol for telling ERC where power comes from"
+			(at 160.02 138.43 0)
+			(effects
+				(font
+					(size 1.27 1.27)
+				)
+				(hide yes)
+			)
+		)
+		(pin "1"
+		)
+		(instances
+			(project ""
+				(path "/5c43024a-135c-49bd-9b6f-adf795041e03"
+					(reference "#FLG02")
+					(unit 1)
+				)
+			)
+		)
+	)
+	(symbol
 		(lib_id "Connector:Conn_01x04_Pin")
 		(at 203.2 69.85 180)
@@
 		(dnp no)
 		(fields_autoplaced yes)
-		(property "Reference" "I2C_skærm_MALE_headers"
+		(property "Reference" "I2C_skærm_FEMALE_4xpin1"
 			(at 204.47 68.5799 0)
 			(effects
@@
 			)
 		)
-		(property "Footprint" ""
+		(property "Footprint" "Connector_PinHeader_2.54mm:PinHeader_1x04_P2.54mm_Vertical"
 			(at 203.2 69.85 0)
 			(effects
@@
 			(project ""
 				(path "/5c43024a-135c-49bd-9b6f-adf795041e03"
-					(reference "I2C_skærm_MALE_headers")
+					(reference "I2C_skærm_FEMALE_4xpin1")
 					(unit 1)
 				)
@@
 	)
 	(symbol
+		(lib_id "power:PWR_FLAG")
+		(at 166.37 125.73 90)
+		(unit 1)
+		(exclude_from_sim no)
+		(in_bom yes)
+		(on_board yes)
+		(dnp no)
+		(property "Reference" "#FLG01"
+			(at 164.465 125.73 0)
+			(effects
+				(font
+					(size 1.27 1.27)
+				)
+				(hide yes)
+			)
+		)
+		(property "Value" "PWR_FLAG"
+			(at 178.816 126.746 90)
+			(effects
+				(font
+					(size 1.27 1.27)
+				)
+				(justify left)
+			)
+		)
+		(property "Footprint" ""
+			(at 166.37 125.73 0)
+			(effects
+				(font
+					(size 1.27 1.27)
+				)
+				(hide yes)
+			)
+		)
+		(property "Datasheet" "~"
+			(at 166.37 125.73 0)
+			(effects
+				(font
+					(size 1.27 1.27)
+				)
+				(hide yes)
+			)
+		)
+		(property "Description" "Special symbol for telling ERC where power comes from"
+			(at 166.37 125.73 0)
+			(effects
+				(font
+					(size 1.27 1.27)
+				)
+				(hide yes)
+			)
+		)
+		(pin "1"
+		)
+		(instances
+			(project ""
+				(path "/5c43024a-135c-49bd-9b6f-adf795041e03"
+					(reference "#FLG01")
+					(unit 1)
+				)
+			)
+		)
+	)
+	(symbol
 		(lib_id "power:GND")
 		(at 120.65 130.81 0)
@@
 			)
 		)
-		(property "Footprint" "Package_DFN_QFN:DFN-8-1EP_3x2mm_P0.5mm_EP1.75x1.45mm"
+		(property "Footprint" "Package_DIP:DIP-8_W7.62mm"
 			(at 144.78 143.51 0)
 			(effects
@@
 		)
 	)
+	(embedded_fonts no)
 )
